File: rp_ext_clk_brd/rp_ext_clk_brd.kicad_pcb (KiCad board)
At the start: 2 copper layers, 43 parts, among them J1 EXT_Connector_2, J2 Screw_Terminal_01x02, J3 EXT_Connector_1, J4 732512120, J5 732512120, U1 SN65LVDT122D, U2 LTC6754HUD-PBF, U3 ADM7171ACPZ-3.3-R7, U4 SN74LVC1G07DBVR, Y1 AK7DAF1-125.0000

Commit message: started routing
Parts:
- added R6: 49.9, Resistor_SMD:R_0603_1608Metric, F.Cu at (230.4, 55.3)
- J1, J3: moved to B.Cu
- J2: value Screw_Terminal_01x02 -> 1860196; footprint TerminalBlock_CUI:TerminalBlock_CUI_TB007-508-02_1x02_P5.08mm_Horizontal -> 1860196:1860196
- J4, J5: value 732512120 -> Conn_Coaxial; footprint Conn_Coax_MLX:CONN-732513152_MOL -> Connector_Coaxial:SMA_Samtec_SMA-J-P-H-ST-EM1_EdgeMount
- moved C1 159.8 mm to (224.0, 69.3)
- moved C13 159.8 mm to (196.0, 71.2)
- moved C14 159.8 mm to (196.0, 73.7)
- moved C17 159.8 mm to (200.0, 66.1)
- moved C18 159.8 mm to (208.8, 66.6)
- moved C19 159.8 mm to (208.8, 69.9)
- moved C2 159.8 mm to (224.0, 72.3)
- moved C21 159.8 mm to (200.0, 68.7)
- moved C24 159.8 mm to (208.8, 73.3)
- moved C7 159.8 mm to (196.0, 66.1)
- moved C8 159.8 mm to (196.0, 68.7)
- moved JP1 159.8 mm to (196.3, 57.5)
- moved JP2 159.8 mm to (200.9, 57.5)
- moved JP3 159.8 mm to (205.4, 57.5)
- moved U3 159.8 mm to (217.1, 52.7)
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Connections:
- C1 pad 1: Net-(J2-Pin_2) -> Net-(U3-EN)
- J2 pad 1: GND -> Net-(U3-EN)
- J2 pad 2: Net-(J2-Pin_2) -> GND
- U1 pad 6: /XTAL_P -> /XTAL_N
- U1 pad 7: /XTAL_N -> /XTAL_P
- U3 pad 5: Net-(J2-Pin_2) -> Net-(U3-EN)
- U3 pad 7: Net-(J2-Pin_2) -> Net-(U3-EN)
- U3 pad 8: Net-(J2-Pin_2) -> Net-(U3-EN)
Routing:
- net /XTAL_P: track 0.00 -> 11.4 mm
- net /XTAL_N: track 0.00 -> 11.4 mm
- net /Q_P: track 0.00 -> 9.17 mm
- net /Q_N: track 0.00 -> 9.17 mm
- net Net-(J4-In): track 0.00 -> 4.46 mm
Other:
- board outline added: 56 x 60 mm
- copper layers 2 -> 4
